File: Design/H00R6.sch (EAGLE design)
At the start: 1 part, among them P1 HEXABIT_17.32

Commit message: -Update the schematic logo
Other:
- note added: "H00R6"
- note added: "H00R6_Frontend"
- note removed: "0"
- note removed: "H00R60"
- note removed: "H00R60_Frontend"
